Commit message: Setup for week 4

File: Creatures/test.urdf (robot description, URDF)
Before this commit: robot rob, 5 links, 4 joints
Links:
- link 0: mass 1.0431724909473667 -> 0.006975861558868622; geometry collision cylinder length=0.08836154654973816 radius=0.1585230194629782; visual cylinder length=0.08836154654973816 radius=0.1585230194629782
- link 11: mass 0.23503100566572174 -> 0.24813741149552138; geometry collision cylinder length=0.13502334083852874 radius=0.7648332547537449; visual cylinder length=0.13502334083852874 radius=0.7648332547537449
- link 12: mass 0.23503100566572174 -> 0.24813741149552138; geometry collision cylinder length=0.13502334083852874 radius=0.7648332547537449; visual cylinder length=0.13502334083852874 radius=0.7648332547537449
- link 13: mass 0.23503100566572174 -> 0.24813741149552138; geometry collision cylinder length=0.13502334083852874 radius=0.7648332547537449; visual cylinder length=0.13502334083852874 radius=0.7648332547537449
- link 24: mass 0.001717621036961022 -> 1.3367442424604354; geometry collision cylinder length=0.5304005544195568 radius=0.8956683750472866; visual cylinder length=0.5304005544195568 radius=0.8956683750472866
Joints:
- joint 11_to_0: axis 0 0 1 -> 1 0 0; origin xyz=0.5790564755296627 0.4578592116065312 0.6232445698945813 rpy=2.151923557371749 4.731704154840095 3.2191729209334317 -> xyz=0.42055318491301796 0.24229778230157661 0.14620923775217187 rpy=4.053520829206385 5.718736773069751 5.552477539633155
- joint 12_to_0: axis 0 0 1 -> 1 0 0; origin xyz=0.5790564755296627 0.4578592116065312 0.6232445698945813 rpy=3.227885336057623 4.731704154840095 3.2191729209334317 -> xyz=0.42055318491301796 0.24229778230157661 0.14620923775217187 rpy=6.080281243809578 5.718736773069751 5.552477539633155
- joint 13_to_0: axis 0 0 1 -> 1 0 0; origin xyz=0.5790564755296627 0.4578592116065312 0.6232445698945813 rpy=4.303847114743498 4.731704154840095 3.2191729209334317 -> xyz=0.42055318491301796 0.24229778230157661 0.14620923775217187 rpy=8.10704165841277 5.718736773069751 5.552477539633155
- joint 24_to_0: origin xyz=0.7571858295084349 0.7047426672682624 0.3740678247259577 rpy=10.510552173729401 2.4501656616869476 4.0557251258886895 -> xyz=0.6013354042847707 0.2677880549967886 0.5853857264131865 rpy=27.345740314979498 3.705843663863804 1.9251116116909397
