Commit message: Multi threaded sim created (mac infinite loop)

File: Creatures/temp.urdf (robot description, URDF)
Before this commit: robot rob, 7 links, 6 joints
Links:
- removed link 14
- removed link 26
- added link 24, mass 0.3450221873082667; collision cylinder length=0.7687676898727434 radius=0.37796450308297536; visual cylinder length=0.7687676898727434 radius=0.37796450308297536
- link 0: mass 0.24005269869841647 -> 0.5408184671904129; geometry collision cylinder length=0.6885731031801839 radius=0.5000066643785868; visual cylinder length=0.6885731031801839 radius=0.5000066643785868
- link 11: mass 1.1963426746848624 -> 1.0538136398121012; geometry collision cylinder length=0.6065321253163667 radius=0.7436696660218431; visual cylinder length=0.6065321253163667 radius=0.7436696660218431
- link 12: mass 1.1963426746848624 -> 1.0538136398121012; geometry collision cylinder length=0.6065321253163667 radius=0.7436696660218431; visual cylinder length=0.6065321253163667 radius=0.7436696660218431
- link 13: mass 1.1963426746848624 -> 1.0538136398121012; geometry collision cylinder length=0.6065321253163667 radius=0.7436696660218431; visual cylinder length=0.6065321253163667 radius=0.7436696660218431
- link 25: mass 0.1221652022463536 -> 0.3450221873082667; geometry collision cylinder length=0.7687676898727434 radius=0.37796450308297536; visual cylinder length=0.7687676898727434 radius=0.37796450308297536
Joints:
- removed joint 14_to_0
- removed joint 26_to_0
- added joint 24_to_0: type revolute, parent 0, child 24, origin xyz=0.33882226597321674 0.3665991098778886 0.8762041938381492 rpy=24.708662815572957 3.5090137775559835 1.4983289205736268, axis 1 0 0, limit lower=3.1415 upper=-3.1415 effort=1 velocity=1
- joint 11_to_0: axis 0 1 0 -> 1 0 0; origin xyz=0.48191692274969455 0.46500400081245785 0.07521811473326923 rpy=1.8511909091374907 5.550839604013139 3.972959372117874 -> xyz=0.9694306409044672 0.7731945385048201 0.9708492058975732 rpy=7.701361495133089 2.8256097181372475 5.943517696791341
- joint 12_to_0: axis 0 1 0 -> 1 0 0; origin xyz=0.48191692274969455 0.46500400081245785 0.07521811473326923 rpy=2.776786363706236 5.550839604013139 3.972959372117874 -> xyz=0.9694306409044672 0.7731945385048201 0.9708492058975732 rpy=11.552042242699633 2.8256097181372475 5.943517696791341
- joint 13_to_0: axis 0 1 0 -> 1 0 0; origin xyz=0.48191692274969455 0.46500400081245785 0.07521811473326923 rpy=3.7023818182749815 5.550839604013139 3.972959372117874 -> xyz=0.9694306409044672 0.7731945385048201 0.9708492058975732 rpy=15.402722990266177 2.8256097181372475 5.943517696791341
- joint 25_to_0: axis 0 1 0 -> 1 0 0; origin xyz=0.2825982067705155 0.5200898462979705 0.023667406151556047 rpy=32.76942761981394 4.1401150230153085 5.711299810008452 -> xyz=0.33882226597321674 0.3665991098778886 0.8762041938381492 rpy=29.65039537868755 3.5090137775559835 1.4983289205736268

File: Creatures/test.urdf (robot description, URDF)
Before this commit: robot rob, 5 links, 4 joints
Links:
- removed link 12
- removed link 13
- removed link 24
- added link 14, mass 0.1672679818027179; collision cylinder length=0.1301162622284413 radius=0.6396842863871616; visual cylinder length=0.1301162622284413 radius=0.6396842863871616
- added link 22, mass 0.4804779648575365; collision cylinder length=0.5004106031336716 radius=0.5528388433329504; visual cylinder length=0.5004106031336716 radius=0.5528388433329504
- added link 23, mass 0.4804779648575365; collision cylinder length=0.5004106031336716 radius=0.5528388433329504; visual cylinder length=0.5004106031336716 radius=0.5528388433329504
- added link 25, mass 0.4804779648575365; collision cylinder length=0.5004106031336716 radius=0.5528388433329504; visual cylinder length=0.5004106031336716 radius=0.5528388433329504
- added link 26, mass 0.4804779648575365; collision cylinder length=0.5004106031336716 radius=0.5528388433329504; visual cylinder length=0.5004106031336716 radius=0.5528388433329504
- link 0: mass 0.006975861558868622 -> 1.3286245026128916; geometry collision cylinder length=0.8311077692460849 radius=0.7133415503554409; visual cylinder length=0.8311077692460849 radius=0.7133415503554409
- link 11: mass 0.24813741149552138 -> 0.1672679818027179; geometry collision cylinder length=0.1301162622284413 radius=0.6396842863871616; visual cylinder length=0.1301162622284413 radius=0.6396842863871616
Joints:
- removed joint 12_to_0
- removed joint 13_to_0
- removed joint 24_to_0
- added joint 14_to_0: type revolute, parent 0, child 14, origin xyz=0.3856918146757604 0.6455790526359318 0.26002697370264016 rpy=10.06388348240069 4.232264990838976 5.462456208406226, axis 0 1 0, limit lower=3.1415 upper=-3.1415 effort=1 velocity=1
- added joint 22_to_11: type revolute, parent 11, child 22, origin xyz=0.7315757928942095 0.9006839698211685 0.15763893767414006 rpy=6.813628014804504 4.754819634558959 2.1685401257119237, axis 1 0 0, limit lower=3.1415 upper=-3.1415 effort=1 velocity=1
- added joint 23_to_11: type revolute, parent 11, child 23, origin xyz=0.7315757928942095 0.9006839698211685 0.15763893767414006 rpy=10.220442022206756 4.754819634558959 2.1685401257119237, axis 1 0 0, limit lower=3.1415 upper=-3.1415 effort=1 velocity=1
- added joint 25_to_14: type revolute, parent 14, child 25, origin xyz=0.7315757928942095 0.9006839698211685 0.15763893767414006 rpy=6.813628014804504 4.754819634558959 2.1685401257119237, axis 1 0 0, limit lower=3.1415 upper=-3.1415 effort=1 velocity=1
- added joint 26_to_14: type revolute, parent 14, child 26, origin xyz=0.7315757928942095 0.9006839698211685 0.15763893767414006 rpy=10.220442022206756 4.754819634558959 2.1685401257119237, axis 1 0 0, limit lower=3.1415 upper=-3.1415 effort=1 velocity=1
- joint 11_to_0: axis 1 0 0 -> 0 1 0; origin xyz=0.42055318491301796 0.24229778230157661 0.14620923775217187 rpy=4.053520829206385 5.718736773069751 5.552477539633155 -> xyz=0.3856918146757604 0.6455790526359318 0.26002697370264016 rpy=6.709255654933793 4.232264990838976 5.462456208406226
