Commit message: Altered for single thread sim

File: Creatures/temp0.urdf (robot description, URDF)
Before this commit: robot pepe, 8 links, 7 joints
Links:
- removed link 24
- removed link 26
- removed link 27
- added link 14, mass 0.9588440740832148; collision cylinder length=0.8655964524447954 radius=0.5938015460244012; visual cylinder length=0.8655964524447954 radius=0.5938015460244012
- link 0: mass 1.9302006588972291 -> 2.316934411795562; geometry collision cylinder length=0.9468658796365681 radius=0.8825467095629808; visual cylinder length=0.9468658796365681 radius=0.8825467095629808
- link 11: mass 0.12838254665197313 -> 0.9588440740832148; geometry collision cylinder length=0.8655964524447954 radius=0.5938015460244012; visual cylinder length=0.8655964524447954 radius=0.5938015460244012
- link 12: mass 0.12838254665197313 -> 0.9588440740832148; geometry collision cylinder length=0.8655964524447954 radius=0.5938015460244012; visual cylinder length=0.8655964524447954 radius=0.5938015460244012
- link 13: mass 0.12838254665197313 -> 0.9588440740832148; geometry collision cylinder length=0.8655964524447954 radius=0.5938015460244012; visual cylinder length=0.8655964524447954 radius=0.5938015460244012
- link 25: mass 0.13544094286480549 -> 1.1071085897364297; geometry collision cylinder length=0.8086510718733262 radius=0.6601453835202641; visual cylinder length=0.8086510718733262 radius=0.6601453835202641
Joints:
- removed joint 24_to_0
- removed joint 26_to_0
- removed joint 27_to_0
- added joint 14_to_0: type revolute, parent 0, child 14, origin xyz=0.044554485920938136 0.023154976680399897 0.8884342370844734 rpy=26.54788508252075 3.9144489454725457 1.238321839973915, axis 0 1 0, limit lower=3.1415 upper=-3.1415 effort=1 velocity=1
- joint 11_to_0: axis 0 0 1 -> 0 1 0; origin xyz=0.18075410986324558 0.318324517345575 0.09242202667278432 rpy=4.768642919376872 1.3159815986997336 3.0551469995826306 -> xyz=0.044554485920938136 0.023154976680399897 0.8884342370844734 rpy=10.6191540330083 3.9144489454725457 1.238321839973915
- joint 12_to_0: axis 0 0 1 -> 0 1 0; origin xyz=0.18075410986324558 0.318324517345575 0.09242202667278432 rpy=7.152964379065308 1.3159815986997336 3.0551469995826306 -> xyz=0.044554485920938136 0.023154976680399897 0.8884342370844734 rpy=15.92873104951245 3.9144489454725457 1.238321839973915
- joint 13_to_0: axis 0 0 1 -> 0 1 0; origin xyz=0.18075410986324558 0.318324517345575 0.09242202667278432 rpy=9.537285838753744 1.3159815986997336 3.0551469995826306 -> xyz=0.044554485920938136 0.023154976680399897 0.8884342370844734 rpy=21.2383080660166 3.9144489454725457 1.238321839973915
- joint 25_to_0: axis 1 0 0 -> 0 1 0; origin xyz=0.15308723840795324 0.3600544427884409 0.48752142522276687 rpy=29.459499919917043 3.881016282437179 1.4882282909109543 -> xyz=0.9850575657269619 0.9290763979916213 0.7419399626130487 rpy=28.381403145241013 1.0528244871783272 5.610370351102431

Commit message: Complete GA with elite examples

File: Creatures/temp0.urdf (robot description, URDF)
Before this commit: robot pepe, 6 links, 5 joints
Links:
- removed link 12
- removed link 14
- removed link 25
- added link 15, mass 0.002082122907049316; collision cylinder length=0.6548837797595078 radius=0.0318123775332233; visual cylinder length=0.6548837797595078 radius=0.0318123775332233
- added link 22, mass 0.07132628116172457; collision cylinder length=0.9751781296241983 radius=0.15258360723808417; visual cylinder length=0.9751781296241983 radius=0.15258360723808417
- added link 24, mass 0.07132628116172457; collision cylinder length=0.9751781296241983 radius=0.15258360723808417; visual cylinder length=0.9751781296241983 radius=0.15258360723808417
- added link 26, mass 0.07132628116172457; collision cylinder length=0.9751781296241983 radius=0.15258360723808417; visual cylinder length=0.9751781296241983 radius=0.15258360723808417
- link 0: mass 2.316934411795562 -> 0.03192563923899716; geometry collision cylinder length=0.9045662752499287 radius=0.10599238596504235; visual cylinder length=0.9045662752499287 radius=0.10599238596504235
- link 11: mass 0.9588440740832148 -> 0.002082122907049316; geometry collision cylinder length=0.6548837797595078 radius=0.0318123775332233; visual cylinder length=0.6548837797595078 radius=0.0318123775332233
- link 13: mass 0.9588440740832148 -> 0.002082122907049316; geometry collision cylinder length=0.6548837797595078 radius=0.0318123775332233; visual cylinder length=0.6548837797595078 radius=0.0318123775332233
Joints:
- removed joint 12_to_0
- removed joint 14_to_0
- removed joint 25_to_0
- added joint 15_to_0: type revolute, parent 0, child 15, origin xyz=0.7382584635277852 0.8811535766403515 0.6031151370398662 rpy=6.330013696424938 3.9804798010911173 0.9419774132799885, axis 1 0 0, limit lower=3.1415 upper=-3.1415 effort=1 velocity=1
- added joint 22_to_11: type revolute, parent 11, child 22, origin xyz=0.3508753140662825 0.14260692267503394 0.6453925831157293 rpy=11.506416440093894 3.066444164091651 3.907328564003008, axis 1 0 0, limit lower=3.1415 upper=-3.1415 effort=1 velocity=1
- added joint 24_to_13: type revolute, parent 13, child 24, origin xyz=0.3508753140662825 0.14260692267503394 0.6453925831157293 rpy=11.506416440093894 3.066444164091651 3.907328564003008, axis 1 0 0, limit lower=3.1415 upper=-3.1415 effort=1 velocity=1
- added joint 26_to_15: type revolute, parent 15, child 26, origin xyz=0.3508753140662825 0.14260692267503394 0.6453925831157293 rpy=11.506416440093894 3.066444164091651 3.907328564003008, axis 1 0 0, limit lower=3.1415 upper=-3.1415 effort=1 velocity=1
- joint 11_to_0: axis 0 1 0 -> 1 0 0; origin xyz=0.044554485920938136 0.023154976680399897 0.8884342370844734 rpy=10.6191540330083 3.9144489454725457 1.238321839973915 -> xyz=0.7382584635277852 0.8811535766403515 0.6031151370398662 rpy=3.165006848212469 3.9804798010911173 0.9419774132799885
- joint 13_to_0: axis 0 1 0 -> 1 0 0; origin xyz=0.044554485920938136 0.023154976680399897 0.8884342370844734 rpy=21.2383080660166 3.9144489454725457 1.238321839973915 -> xyz=0.7382584635277852 0.8811535766403515 0.6031151370398662 rpy=4.747510272318704 3.9804798010911173 0.9419774132799885

File: Creatures/test.urdf (robot description, URDF)
Before this commit: robot rob, 7 links, 6 joints
Links:
- removed link 14
- removed link 23
- removed link 25
- added link 13, mass 0.002082122907049316; collision cylinder length=0.6548837797595078 radius=0.0318123775332233; visual cylinder length=0.6548837797595078 radius=0.0318123775332233
- added link 15, mass 0.002082122907049316; collision cylinder length=0.6548837797595078 radius=0.0318123775332233; visual cylinder length=0.6548837797595078 radius=0.0318123775332233
- added link 24, mass 0.07132628116172457; collision cylinder length=0.9751781296241983 radius=0.15258360723808417; visual cylinder length=0.9751781296241983 radius=0.15258360723808417
- link 0: mass 1.3286245026128916 -> 0.03192563923899716; geometry collision cylinder length=0.9045662752499287 radius=0.10599238596504235; visual cylinder length=0.9045662752499287 radius=0.10599238596504235
- link 11: mass 0.1672679818027179 -> 0.002082122907049316; geometry collision cylinder length=0.6548837797595078 radius=0.0318123775332233; visual cylinder length=0.6548837797595078 radius=0.0318123775332233
- link 22: mass 0.4804779648575365 -> 0.07132628116172457; geometry collision cylinder length=0.9751781296241983 radius=0.15258360723808417; visual cylinder length=0.9751781296241983 radius=0.15258360723808417
- link 26: mass 0.4804779648575365 -> 0.07132628116172457; geometry collision cylinder length=0.9751781296241983 radius=0.15258360723808417; visual cylinder length=0.9751781296241983 radius=0.15258360723808417
Joints:
- removed joint 14_to_0
- removed joint 23_to_11
- removed joint 25_to_14
- removed joint 26_to_14
- added joint 13_to_0: type revolute, parent 0, child 13, origin xyz=0.7382584635277852 0.8811535766403515 0.6031151370398662 rpy=4.747510272318704 3.9804798010911173 0.9419774132799885, axis 1 0 0, limit lower=3.1415 upper=-3.1415 effort=1 velocity=1
- added joint 15_to_0: type revolute, parent 0, child 15, origin xyz=0.7382584635277852 0.8811535766403515 0.6031151370398662 rpy=6.330013696424938 3.9804798010911173 0.9419774132799885, axis 1 0 0, limit lower=3.1415 upper=-3.1415 effort=1 velocity=1
- added joint 24_to_13: type revolute, parent 13, child 24, origin xyz=0.3508753140662825 0.14260692267503394 0.6453925831157293 rpy=11.506416440093894 3.066444164091651 3.907328564003008, axis 1 0 0, limit lower=3.1415 upper=-3.1415 effort=1 velocity=1
- added joint 26_to_15: type revolute, parent 15, child 26, origin xyz=0.3508753140662825 0.14260692267503394 0.6453925831157293 rpy=11.506416440093894 3.066444164091651 3.907328564003008, axis 1 0 0, limit lower=3.1415 upper=-3.1415 effort=1 velocity=1
- joint 11_to_0: axis 0 1 0 -> 1 0 0; origin xyz=0.3856918146757604 0.6455790526359318 0.26002697370264016 rpy=6.709255654933793 4.232264990838976 5.462456208406226 -> xyz=0.7382584635277852 0.8811535766403515 0.6031151370398662 rpy=3.165006848212469 3.9804798010911173 0.9419774132799885
- joint 22_to_11: origin xyz=0.7315757928942095 0.9006839698211685 0.15763893767414006 rpy=6.813628014804504 4.754819634558959 2.1685401257119237 -> xyz=0.3508753140662825 0.14260692267503394 0.6453925831157293 rpy=11.506416440093894 3.066444164091651 3.907328564003008
