Commit message: Prep for robot scientist

File: Creatures/temp0.urdf (robot description, URDF)
Before this commit: robot pepe, 7 links, 6 joints
Links:
- removed link 13
- removed link 15
- removed link 24
- removed link 26
- added link 110, mass 0.010253105311762557; collision cylinder length=0.6554050905461422 radius=0.07056638464046394; visual cylinder length=0.6554050905461422 radius=0.07056638464046394
- added link 119, mass 0.010253105311762557; collision cylinder length=0.6554050905461422 radius=0.07056638464046394; visual cylinder length=0.6554050905461422 radius=0.07056638464046394
- added link 211, mass 0.06800321921601057; collision cylinder length=0.9825247934196826 radius=0.14842875362748054; visual cylinder length=0.9825247934196826 radius=0.14842875362748054
- added link 212, mass 0.06800321921601057; collision cylinder length=0.9825247934196826 radius=0.14842875362748054; visual cylinder length=0.9825247934196826 radius=0.14842875362748054
- added link 220, mass 0.06800321921601057; collision cylinder length=0.9825247934196826 radius=0.14842875362748054; visual cylinder length=0.9825247934196826 radius=0.14842875362748054
- added link 221, mass 0.06800321921601057; collision cylinder length=0.9825247934196826 radius=0.14842875362748054; visual cylinder length=0.9825247934196826 radius=0.14842875362748054
- added link 23, mass 0.06800321921601057; collision cylinder length=0.9825247934196826 radius=0.14842875362748054; visual cylinder length=0.9825247934196826 radius=0.14842875362748054
- added link 313, mass 0.16743777760307593; collision cylinder length=0.21221130422533313 radius=0.501149765989212; visual cylinder length=0.21221130422533313 radius=0.501149765989212
- added link 314, mass 0.16743777760307593; collision cylinder length=0.21221130422533313 radius=0.501149765989212; visual cylinder length=0.21221130422533313 radius=0.501149765989212
- added link 315, mass 0.16743777760307593; collision cylinder length=0.21221130422533313 radius=0.501149765989212; visual cylinder length=0.21221130422533313 radius=0.501149765989212
- added link 322, mass 0.16743777760307593; collision cylinder length=0.21221130422533313 radius=0.501149765989212; visual cylinder length=0.21221130422533313 radius=0.501149765989212
- added link 323, mass 0.16743777760307593; collision cylinder length=0.21221130422533313 radius=0.501149765989212; visual cylinder length=0.21221130422533313 radius=0.501149765989212
- added link 324, mass 0.16743777760307593; collision cylinder length=0.21221130422533313 radius=0.501149765989212; visual cylinder length=0.21221130422533313 radius=0.501149765989212
- added link 34, mass 0.16743777760307593; collision cylinder length=0.21221130422533313 radius=0.501149765989212; visual cylinder length=0.21221130422533313 radius=0.501149765989212
- added link 35, mass 0.16743777760307593; collision cylinder length=0.21221130422533313 radius=0.501149765989212; visual cylinder length=0.21221130422533313 radius=0.501149765989212
- added link 36, mass 0.16743777760307593; collision cylinder length=0.21221130422533313 radius=0.501149765989212; visual cylinder length=0.21221130422533313 radius=0.501149765989212
- added link 416, mass 0.027705168971618666; collision cylinder length=0.9225313326126843 radius=0.09777209083909966; visual cylinder length=0.9225313326126843 radius=0.09777209083909966
- added link 417, mass 0.027705168971618666; collision cylinder length=0.9225313326126843 radius=0.09777209083909966; visual cylinder length=0.9225313326126843 radius=0.09777209083909966
- added link 418, mass 0.027705168971618666; collision cylinder length=0.9225313326126843 radius=0.09777209083909966; visual cylinder length=0.9225313326126843 radius=0.09777209083909966
- added link 425, mass 0.027705168971618666; collision cylinder length=0.9225313326126843 radius=0.09777209083909966; visual cylinder length=0.9225313326126843 radius=0.09777209083909966
- added link 426, mass 0.027705168971618666; collision cylinder length=0.9225313326126843 radius=0.09777209083909966; visual cylinder length=0.9225313326126843 radius=0.09777209083909966
- added link 427, mass 0.027705168971618666; collision cylinder length=0.9225313326126843 radius=0.09777209083909966; visual cylinder length=0.9225313326126843 radius=0.09777209083909966
- added link 47, mass 0.027705168971618666; collision cylinder length=0.9225313326126843 radius=0.09777209083909966; visual cylinder length=0.9225313326126843 radius=0.09777209083909966
- added link 48, mass 0.027705168971618666; collision cylinder length=0.9225313326126843 radius=0.09777209083909966; visual cylinder length=0.9225313326126843 radius=0.09777209083909966
- added link 49, mass 0.027705168971618666; collision cylinder length=0.9225313326126843 radius=0.09777209083909966; visual cylinder length=0.9225313326126843 radius=0.09777209083909966
- link 0: mass 0.03192563923899716 -> 0.033545493768338736; geometry collision cylinder length=0.293104550776125 radius=0.1908670131524005; visual cylinder length=0.293104550776125 radius=0.1908670131524005
- link 11: mass 0.002082122907049316 -> 0.010253105311762557; geometry collision cylinder length=0.6554050905461422 radius=0.07056638464046394; visual cylinder length=0.6554050905461422 radius=0.07056638464046394
- link 22: mass 0.07132628116172457 -> 0.06800321921601057; geometry collision cylinder length=0.9825247934196826 radius=0.14842875362748054; visual cylinder length=0.9825247934196826 radius=0.14842875362748054
Joints:
- removed joint 13_to_0
- removed joint 15_to_0
- removed joint 24_to_13
- removed joint 26_to_15
- added joint 110_to_0: type revolute, parent 0, child 110, origin xyz=0.16753311632188983 0.36515283006603405 0.7821485066599133 rpy=3.5433921955531344 4.758617516157513 3.1710336822631713, axis 1 0 0, limit lower=3.1415 upper=-3.1415 effort=1 velocity=1
- added joint 119_to_0: type revolute, parent 0, child 119, origin xyz=0.16753311632188983 0.36515283006603405 0.7821485066599133 rpy=4.72452292740418 4.758617516157513 3.1710336822631713, axis 1 0 0, limit lower=3.1415 upper=-3.1415 effort=1 velocity=1
- added joint 211_to_110: type revolute, parent 110, child 211, origin xyz=0.04663399306933716 0.5685102803336283 0.055749497347352794 rpy=11.417892777568959 1.9775569174688448 5.724771741504134, axis 1 0 0, limit lower=3.1415 upper=-3.1415 effort=1 velocity=1
- added joint 212_to_110: type revolute, parent 110, child 212, origin xyz=0.04663399306933716 0.5685102803336283 0.055749497347352794 rpy=17.126839166353438 1.9775569174688448 5.724771741504134, axis 1 0 0, limit lower=3.1415 upper=-3.1415 effort=1 velocity=1
- added joint 220_to_119: type revolute, parent 119, child 220, origin xyz=0.04663399306933716 0.5685102803336283 0.055749497347352794 rpy=11.417892777568959 1.9775569174688448 5.724771741504134, axis 1 0 0, limit lower=3.1415 upper=-3.1415 effort=1 velocity=1
- added joint 221_to_119: type revolute, parent 119, child 221, origin xyz=0.04663399306933716 0.5685102803336283 0.055749497347352794 rpy=17.126839166353438 1.9775569174688448 5.724771741504134, axis 1 0 0, limit lower=3.1415 upper=-3.1415 effort=1 velocity=1
- added joint 23_to_11: type revolute, parent 11, child 23, origin xyz=0.04663399306933716 0.5685102803336283 0.055749497347352794 rpy=17.126839166353438 1.9775569174688448 5.724771741504134, axis 1 0 0, limit lower=3.1415 upper=-3.1415 effort=1 velocity=1
- added joint 313_to_110: type revolute, parent 110, child 313, origin xyz=0.5427969302190827 -0.00926040214177129 -0.03423992650931537 rpy=21.29865546162663 5.432332058375099 1.8074472366872858, axis 1 0 0, limit lower=3.1415 upper=-3.1415 effort=1 velocity=1
- added joint 314_to_110: type revolute, parent 110, child 314, origin xyz=0.5427969302190827 -0.00926040214177129 -0.03423992650931537 rpy=26.623319327033286 5.432332058375099 1.8074472366872858, axis 1 0 0, limit lower=3.1415 upper=-3.1415 effort=1 velocity=1
- added joint 315_to_110: type revolute, parent 110, child 315, origin xyz=0.5427969302190827 -0.00926040214177129 -0.03423992650931537 rpy=31.947983192439946 5.432332058375099 1.8074472366872858, axis 1 0 0, limit lower=3.1415 upper=-3.1415 effort=1 velocity=1
- added joint 322_to_119: type revolute, parent 119, child 322, origin xyz=0.5427969302190827 -0.00926040214177129 -0.03423992650931537 rpy=21.29865546162663 5.432332058375099 1.8074472366872858, axis 1 0 0, limit lower=3.1415 upper=-3.1415 effort=1 velocity=1
- added joint 323_to_119: type revolute, parent 119, child 323, origin xyz=0.5427969302190827 -0.00926040214177129 -0.03423992650931537 rpy=26.623319327033286 5.432332058375099 1.8074472366872858, axis 1 0 0, limit lower=3.1415 upper=-3.1415 effort=1 velocity=1
- added joint 324_to_119: type revolute, parent 119, child 324, origin xyz=0.5427969302190827 -0.00926040214177129 -0.03423992650931537 rpy=31.947983192439946 5.432332058375099 1.8074472366872858, axis 1 0 0, limit lower=3.1415 upper=-3.1415 effort=1 velocity=1
- added joint 34_to_11: type revolute, parent 11, child 34, origin xyz=0.5427969302190827 -0.00926040214177129 -0.03423992650931537 rpy=21.29865546162663 5.432332058375099 1.8074472366872858, axis 1 0 0, limit lower=3.1415 upper=-3.1415 effort=1 velocity=1
- added joint 35_to_11: type revolute, parent 11, child 35, origin xyz=0.5427969302190827 -0.00926040214177129 -0.03423992650931537 rpy=26.623319327033286 5.432332058375099 1.8074472366872858, axis 1 0 0, limit lower=3.1415 upper=-3.1415 effort=1 velocity=1
- added joint 36_to_11: type revolute, parent 11, child 36, origin xyz=0.5427969302190827 -0.00926040214177129 -0.03423992650931537 rpy=31.947983192439946 5.432332058375099 1.8074472366872858, axis 1 0 0, limit lower=3.1415 upper=-3.1415 effort=1 velocity=1
- added joint 416_to_110: type revolute, parent 110, child 416, origin xyz=0.684706195222893 0.8600171314791502 0.5770014648713004 rpy=16.812008871190226 2.187456646668616 3.8407791478327677, axis 1 0 0, limit lower=3.1415 upper=-3.1415 effort=1 velocity=1
- added joint 417_to_110: type revolute, parent 110, child 417, origin xyz=0.684706195222893 0.8600171314791502 0.5770014648713004 rpy=19.2137244242174 2.187456646668616 3.8407791478327677, axis 1 0 0, limit lower=3.1415 upper=-3.1415 effort=1 velocity=1
- added joint 418_to_110: type revolute, parent 110, child 418, origin xyz=0.684706195222893 0.8600171314791502 0.5770014648713004 rpy=21.615439977244574 2.187456646668616 3.8407791478327677, axis 1 0 0, limit lower=3.1415 upper=-3.1415 effort=1 velocity=1
- added joint 425_to_119: type revolute, parent 119, child 425, origin xyz=0.684706195222893 0.8600171314791502 0.5770014648713004 rpy=16.812008871190226 2.187456646668616 3.8407791478327677, axis 1 0 0, limit lower=3.1415 upper=-3.1415 effort=1 velocity=1
- added joint 426_to_119: type revolute, parent 119, child 426, origin xyz=0.684706195222893 0.8600171314791502 0.5770014648713004 rpy=19.2137244242174 2.187456646668616 3.8407791478327677, axis 1 0 0, limit lower=3.1415 upper=-3.1415 effort=1 velocity=1
- added joint 427_to_119: type revolute, parent 119, child 427, origin xyz=0.684706195222893 0.8600171314791502 0.5770014648713004 rpy=21.615439977244574 2.187456646668616 3.8407791478327677, axis 1 0 0, limit lower=3.1415 upper=-3.1415 effort=1 velocity=1
- added joint 47_to_11: type revolute, parent 11, child 47, origin xyz=0.684706195222893 0.8600171314791502 0.5770014648713004 rpy=16.812008871190226 2.187456646668616 3.8407791478327677, axis 1 0 0, limit lower=3.1415 upper=-3.1415 effort=1 velocity=1
- added joint 48_to_11: type revolute, parent 11, child 48, origin xyz=0.684706195222893 0.8600171314791502 0.5770014648713004 rpy=19.2137244242174 2.187456646668616 3.8407791478327677, axis 1 0 0, limit lower=3.1415 upper=-3.1415 effort=1 velocity=1
- added joint 49_to_11: type revolute, parent 11, child 49, origin xyz=0.684706195222893 0.8600171314791502 0.5770014648713004 rpy=21.615439977244574 2.187456646668616 3.8407791478327677, axis 1 0 0, limit lower=3.1415 upper=-3.1415 effort=1 velocity=1
- joint 11_to_0: origin xyz=0.7382584635277852 0.8811535766403515 0.6031151370398662 rpy=3.165006848212469 3.9804798010911173 0.9419774132799885 -> xyz=0.16753311632188983 0.36515283006603405 0.7821485066599133 rpy=2.36226146370209 4.758617516157513 3.1710336822631713
- joint 22_to_11: origin xyz=0.3508753140662825 0.14260692267503394 0.6453925831157293 rpy=11.506416440093894 3.066444164091651 3.907328564003008 -> xyz=0.04663399306933716 0.5685102803336283 0.055749497347352794 rpy=11.417892777568959 1.9775569174688448 5.724771741504134

File: Creatures/test.urdf (robot description, URDF)
Before this commit: robot pepe, 7 links, 6 joints
Links:
- removed link 13
- removed link 15
- removed link 24
- removed link 26
- added link 113, mass 0.010253105311762557; collision cylinder length=0.6554050905461422 radius=0.07056638464046394; visual cylinder length=0.6554050905461422 radius=0.07056638464046394
- added link 17, mass 0.010253105311762557; collision cylinder length=0.6554050905461422 radius=0.07056638464046394; visual cylinder length=0.6554050905461422 radius=0.07056638464046394
- added link 214, mass 0.09182745029567585; collision cylinder length=0.9825247934196826 radius=0.17248032719250542; visual cylinder length=0.9825247934196826 radius=0.17248032719250542
- added link 215, mass 0.09182745029567585; collision cylinder length=0.9825247934196826 radius=0.17248032719250542; visual cylinder length=0.9825247934196826 radius=0.17248032719250542
- added link 23, mass 0.09182745029567585; collision cylinder length=0.9825247934196826 radius=0.17248032719250542; visual cylinder length=0.9825247934196826 radius=0.17248032719250542
- added link 28, mass 0.09182745029567585; collision cylinder length=0.9825247934196826 radius=0.17248032719250542; visual cylinder length=0.9825247934196826 radius=0.17248032719250542
- added link 29, mass 0.09182745029567585; collision cylinder length=0.9825247934196826 radius=0.17248032719250542; visual cylinder length=0.9825247934196826 radius=0.17248032719250542
- added link 310, mass 0.16743777760307593; collision cylinder length=0.21221130422533313 radius=0.501149765989212; visual cylinder length=0.21221130422533313 radius=0.501149765989212
- added link 311, mass 0.16743777760307593; collision cylinder length=0.21221130422533313 radius=0.501149765989212; visual cylinder length=0.21221130422533313 radius=0.501149765989212
- added link 312, mass 0.16743777760307593; collision cylinder length=0.21221130422533313 radius=0.501149765989212; visual cylinder length=0.21221130422533313 radius=0.501149765989212
- added link 316, mass 0.16743777760307593; collision cylinder length=0.21221130422533313 radius=0.501149765989212; visual cylinder length=0.21221130422533313 radius=0.501149765989212
- added link 317, mass 0.16743777760307593; collision cylinder length=0.21221130422533313 radius=0.501149765989212; visual cylinder length=0.21221130422533313 radius=0.501149765989212
- added link 318, mass 0.16743777760307593; collision cylinder length=0.21221130422533313 radius=0.501149765989212; visual cylinder length=0.21221130422533313 radius=0.501149765989212
- added link 34, mass 0.16743777760307593; collision cylinder length=0.21221130422533313 radius=0.501149765989212; visual cylinder length=0.21221130422533313 radius=0.501149765989212
- added link 35, mass 0.16743777760307593; collision cylinder length=0.21221130422533313 radius=0.501149765989212; visual cylinder length=0.21221130422533313 radius=0.501149765989212
- added link 36, mass 0.16743777760307593; collision cylinder length=0.21221130422533313 radius=0.501149765989212; visual cylinder length=0.21221130422533313 radius=0.501149765989212
- link 0: mass 0.03192563923899716 -> 0.033545493768338736; geometry collision cylinder length=0.293104550776125 radius=0.1908670131524005; visual cylinder length=0.293104550776125 radius=0.1908670131524005
- link 11: mass 0.002082122907049316 -> 0.010253105311762557; geometry collision cylinder length=0.6554050905461422 radius=0.07056638464046394; visual cylinder length=0.6554050905461422 radius=0.07056638464046394
- link 22: mass 0.07132628116172457 -> 0.09182745029567585; geometry collision cylinder length=0.9825247934196826 radius=0.17248032719250542; visual cylinder length=0.9825247934196826 radius=0.17248032719250542
Joints:
- removed joint 13_to_0
- removed joint 15_to_0
- removed joint 24_to_13
- removed joint 26_to_15
- added joint 113_to_0: type revolute, parent 0, child 113, origin xyz=0.16753311632188983 0.36515283006603405 0.7821485066599133 rpy=4.72452292740418 4.758617516157513 3.1710336822631713, axis 1 0 0, limit lower=3.1415 upper=-3.1415 effort=1 velocity=1
- added joint 17_to_0: type revolute, parent 0, child 17, origin xyz=0.16753311632188983 0.36515283006603405 0.7821485066599133 rpy=3.5433921955531344 4.758617516157513 3.1710336822631713, axis 1 0 0, limit lower=3.1415 upper=-3.1415 effort=1 velocity=1
- added joint 214_to_113: type revolute, parent 113, child 214, origin xyz=0.04663399306933716 0.47766581814305353 0.055749497347352794 rpy=11.417892777568959 1.9775569174688448 5.724771741504134, axis 1 0 0, limit lower=3.1415 upper=-3.1415 effort=1 velocity=1
- added joint 215_to_113: type revolute, parent 113, child 215, origin xyz=0.04663399306933716 0.47766581814305353 0.055749497347352794 rpy=17.126839166353438 1.9775569174688448 5.724771741504134, axis 1 0 0, limit lower=3.1415 upper=-3.1415 effort=1 velocity=1
- added joint 23_to_11: type revolute, parent 11, child 23, origin xyz=0.04663399306933716 0.47766581814305353 0.055749497347352794 rpy=17.126839166353438 1.9775569174688448 5.724771741504134, axis 1 0 0, limit lower=3.1415 upper=-3.1415 effort=1 velocity=1
- added joint 28_to_17: type revolute, parent 17, child 28, origin xyz=0.04663399306933716 0.47766581814305353 0.055749497347352794 rpy=11.417892777568959 1.9775569174688448 5.724771741504134, axis 1 0 0, limit lower=3.1415 upper=-3.1415 effort=1 velocity=1
- added joint 29_to_17: type revolute, parent 17, child 29, origin xyz=0.04663399306933716 0.47766581814305353 0.055749497347352794 rpy=17.126839166353438 1.9775569174688448 5.724771741504134, axis 1 0 0, limit lower=3.1415 upper=-3.1415 effort=1 velocity=1
- added joint 310_to_17: type revolute, parent 17, child 310, origin xyz=0.5427969302190827 -0.00926040214177129 -0.03423992650931537 rpy=21.29865546162663 5.432332058375099 1.8074472366872858, axis 1 0 0, limit lower=3.1415 upper=-3.1415 effort=1 velocity=1
- added joint 311_to_17: type revolute, parent 17, child 311, origin xyz=0.5427969302190827 -0.00926040214177129 -0.03423992650931537 rpy=26.623319327033286 5.432332058375099 1.8074472366872858, axis 1 0 0, limit lower=3.1415 upper=-3.1415 effort=1 velocity=1
- added joint 312_to_17: type revolute, parent 17, child 312, origin xyz=0.5427969302190827 -0.00926040214177129 -0.03423992650931537 rpy=31.947983192439946 5.432332058375099 1.8074472366872858, axis 1 0 0, limit lower=3.1415 upper=-3.1415 effort=1 velocity=1
- added joint 316_to_113: type revolute, parent 113, child 316, origin xyz=0.5427969302190827 -0.00926040214177129 -0.03423992650931537 rpy=21.29865546162663 5.432332058375099 1.8074472366872858, axis 1 0 0, limit lower=3.1415 upper=-3.1415 effort=1 velocity=1
- added joint 317_to_113: type revolute, parent 113, child 317, origin xyz=0.5427969302190827 -0.00926040214177129 -0.03423992650931537 rpy=26.623319327033286 5.432332058375099 1.8074472366872858, axis 1 0 0, limit lower=3.1415 upper=-3.1415 effort=1 velocity=1
- added joint 318_to_113: type revolute, parent 113, child 318, origin xyz=0.5427969302190827 -0.00926040214177129 -0.03423992650931537 rpy=31.947983192439946 5.432332058375099 1.8074472366872858, axis 1 0 0, limit lower=3.1415 upper=-3.1415 effort=1 velocity=1
- added joint 34_to_11: type revolute, parent 11, child 34, origin xyz=0.5427969302190827 -0.00926040214177129 -0.03423992650931537 rpy=21.29865546162663 5.432332058375099 1.8074472366872858, axis 1 0 0, limit lower=3.1415 upper=-3.1415 effort=1 velocity=1
- added joint 35_to_11: type revolute, parent 11, child 35, origin xyz=0.5427969302190827 -0.00926040214177129 -0.03423992650931537 rpy=26.623319327033286 5.432332058375099 1.8074472366872858, axis 1 0 0, limit lower=3.1415 upper=-3.1415 effort=1 velocity=1
- added joint 36_to_11: type revolute, parent 11, child 36, origin xyz=0.5427969302190827 -0.00926040214177129 -0.03423992650931537 rpy=31.947983192439946 5.432332058375099 1.8074472366872858, axis 1 0 0, limit lower=3.1415 upper=-3.1415 effort=1 velocity=1
- joint 11_to_0: origin xyz=0.7382584635277852 0.8811535766403515 0.6031151370398662 rpy=3.165006848212469 3.9804798010911173 0.9419774132799885 -> xyz=0.16753311632188983 0.36515283006603405 0.7821485066599133 rpy=2.36226146370209 4.758617516157513 3.1710336822631713
- joint 22_to_11: origin xyz=0.3508753140662825 0.14260692267503394 0.6453925831157293 rpy=11.506416440093894 3.066444164091651 3.907328564003008 -> xyz=0.04663399306933716 0.47766581814305353 0.055749497347352794 rpy=11.417892777568959 1.9775569174688448 5.724771741504134
